Commit message: feat: move camera for benchmark

File: urdf/camera.xacro (robot description, xacro)
@@ -31,5 +31,5 @@
         <parent link="base_link"/>
         <child link="camera_link"/>
-        <origin xyz="0.5 0 1.2" rpy="0 1.57 0" />
+        <origin xyz="1 0 1.2" rpy="0 1.57 0" />
     </joint>
     <link name="camera_optical_link"></link>
